File: hardware/convert_folder/sources/flatsat_platform_2.kicad_pcb (KiCad board)
At the start: 4 copper layers, 400 x 250 mm, 149 parts, among them CN1 5-146285-2, CN10 5-146285-2, CN13 4243-0, CN14 TSW-101-05-T-S, CN15 JST 2 position header 2.5mm, CN16 JST 2 position header 2.5mm, CN2 4243-0, CN20 PC104_inverted, CN21 PC104, CN22 PC104, CN23 PC104, CN24 PC104, CN25 PC104, CN26 JST 2 position header 2.5mm, CN3 4 pin Picoblade, CN4 6 pin Picoblade, CN5 6 pin Picoblade, CN6 4 pin Picoblade, CN8 5-146285-2, CN9 5-146285-2, IC1 TPS74401RGWRM3, IC2 TPS74401RGWRM3, IC4 TPS3899DL30DSER, IC5 LM321LVIDBVR, IC6 MMBT3904, IC7 MMBT3904, J1 5-146280-2, J10 Soquete de termopar, J11 Soquete de termopar, J12 Soquete de termopar, J13 Soquete de termopar, J14 Soquete de termopar, J15 Soquete de termopar, J2 5-146280-2, J3 1054500101, J4 87832-1420, J5 Soquete de termopar, J6 Soquete de termopar, J8 87832-1420, J9 87832-1420, SW1 434123050836, SW2 SW-T3-2B-A-A3-S1, SW3 SW-T3-2B-A-A3-S1, U1 INA219AID, U12 INA219AID, U13 INA219AID, U18 INA219AID, U19 TMP112AIDRLT, U21 LTC2983CLX#PBF, U22 ISL83483IBZ, U23 SN65HVD232D, U24 SN65HVD232D, U25 ISL83483IBZ, U4 INA219AID, U7 INA219AID, U9 INA219AID

Commit message: fix: start fixing the power converters of the board
Parts:
- added MEC1: M3, altium_import:M3 HOLE, F.Cu at (98.6, 316.1)
- moved MEC2 19.2 mm to (490.6, 74.6)
- moved MEC8 13.1 mm to (98.6, 74.4)
- moved MEC1 8.97 mm to (490.3, 316.1)
Routing:
- net GND: vias 7675 -> 3249
