File: hardware/convert_folder/sources/flatsat_platform_2.kicad_pcb (KiCad board)
At the start: 4 copper layers, 400 x 250 mm, 194 parts, among them CN1 5-146285-2, CN11 5-146285-2, CN13 4243-0, CN15 JST 2 position header 2.5mm, CN2 4243-0, CN20 PC104_inverted, CN21 PC104, CN22 PC104, CN23 PC104, CN24 PC104, CN25 PC104, CN26 JST 2 position header 2.5mm, CN3 4 pin Picoblade, CN4 6 pin Picoblade, CN5 6 pin Picoblade, CN6 4 pin Picoblade, CN7 5-146285-2, CN8 5-146285-2, CN9 5-146285-2, IC1 TPS3780BDBVT, IC2 TPS74401RGWRM3, IC3 TPS74401RGWRM3, IC6 MMBT3904, IC66 TPS74401RGWRM3, IC7 MMBT3904, IC8 TPS74401RGWRM3, J1 5-146280-2, J16 5-146280-2, J17 5-146280-2, J18 5-146280-2, J2 5-146280-2, J3 1054500101, J4 87832-1420, J7 5-146280-2, J8 87832-1420, J9 87832-1420, Q1 BSS138, Q2 BSS138, Q3 BSS138, Q4 BSS138, SW1 SW-T3-2B-A-A3-S1, SW2 SW-T3-2B-A-A3-S1, SW3 SW-T3-2B-A-A3-S1, U1 INA219AID, U12 INA219AID, U13 INA219AID, U18 INA219AID, U19 TMP112AIDRLT, U21 LTC2983CLX#PBF, U22 THVD1450DR, U23 SN65HVD232D, U24 SN65HVD232D, U25 THVD1450DR, U4 INA219AID, U7 INA219AID, U9 INA219AID

Commit message: fix: fix position of components and signals routing
Parts:
- removed J4: 87832-1420, altium_import:SAMTEC_TSW-107-05-F-D
- added J20: 61201421621, lib:61201421621, F.Cu at (333.7, 313.4)
- added J21: 61201421621, lib:61201421621, F.Cu at (333.7, 302.5)
- moved CN15 7.01 mm to (314.6, 311.0)
- moved CN26 7.01 mm to (297.6, 311.0)
- moved CN3 7.01 mm to (314.6, 315.4)
- moved CN6 7.01 mm to (297.3, 315.4)
- moved R47 5.36 mm to (263.3, 260.5)
- moved R40 4.03 mm to (263.3, 305.0)
- moved U22 2.45 mm to (266.8, 311.6)
- moved U25 2.45 mm to (249.4, 311.9)
- moved R46 1.75 mm to (271.9, 283.1)
- moved R45 1.17 mm to (271.9, 284.7)
- moved R160 0.58 mm to (271.9, 286.4)
Routing:
- net /microzed/PL_B13_2N: track 0.00 -> 190.3 mm, vias 0 -> 2
- net /SDA_CHN_1: track 760.3 -> 948.8 mm, vias 8 -> 9
- net /microzed/PL_B13_2P: track 0.00 -> 185.9 mm, vias 0 -> 2
- net /microzed/PL_JX2_14N: track 0.00 -> 183.3 mm, vias 0 -> 2
- net /microzed/PL_JX2_14P: track 0.00 -> 180.8 mm, vias 0 -> 2
- net /microzed/PL_JX2_12N: track 0.00 -> 179.8 mm, vias 0 -> 2
- net /microzed/PL_JX2_12P: track 0.00 -> 177.3 mm, vias 0 -> 2
- net /SCL_CHN_1: track 760.8 -> 913.3 mm, vias 8 -> 9
- net /microzed/<NO NET>: track 0.00 -> 109.8 mm
- net /microzed/PL_JX2_15N: track 0.00 -> 109.6 mm
- net /microzed/PL_JX2_15P: track 0.00 -> 108.8 mm
- net /microzed/PL_JX2_13N: track 0.00 -> 108.6 mm
- net /microzed/PL_JX2_13P: track 0.00 -> 107.8 mm
- net /microzed/PL_B13_6N: track 0.00 -> 103.6 mm, vias 0 -> 1
- net /TX_CHN_4: track 1.40 -> 86.5 mm
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