File: hardware/convert_folder/sources/flatsat_platform_2.kicad_pcb (KiCad board)
At the start: 4 copper layers, 400 x 250 mm, 195 parts, among them CN1 5-146285-2, CN11 5-146285-2, CN13 4243-0, CN15 JST 2 position header 2.5mm, CN2 4243-0, CN20 PC104_inverted, CN21 PC104, CN22 PC104, CN23 PC104, CN24 PC104, CN25 PC104, CN26 JST 2 position header 2.5mm, CN3 4 pin Picoblade, CN4 6 pin Picoblade, CN5 6 pin Picoblade, CN6 4 pin Picoblade, CN7 5-146285-2, CN8 5-146285-2, CN9 5-146285-2, IC1 TPS3780BDBVT, IC2 TPS74401RGWRM3, IC3 TPS74401RGWRM3, IC6 MMBT3904, IC66 TPS74401RGWRM3, IC7 MMBT3904, IC8 TPS74401RGWRM3, J1 5-146280-2, J16 5-146280-2, J17 5-146280-2, J18 5-146280-2, J2 5-146280-2, J20 61201421621, J21 61201421621, J3 1054500101, J7 5-146280-2, J8 87832-1420, J9 87832-1420, Q1 BSS138, Q2 BSS138, Q3 BSS138, Q4 BSS138, SW1 SW-T3-2B-A-A3-S1, SW2 SW-T3-2B-A-A3-S1, SW3 SW-T3-2B-A-A3-S1, U1 INA219AID, U12 INA219AID, U13 INA219AID, U18 INA219AID, U19 TMP112AIDRLT, U21 LTC2983CLX#PBF, U22 THVD1450DR, U23 SN65HVD232D, U24 SN65HVD232D, U25 THVD1450DR, U4 INA219AID, U7 INA219AID, U9 INA219AID

Commit message: fix: minor corrections at the TPS3780 circuit
Parts:
- moved FD7 4.88 mm to (121.7, 204.0)
- moved CN20 0.05 mm to (108.7, 194.8)
Connections:
- net /EPS_H1-46 renamed /EPS_H1-45
- net /EPS_H1-50 renamed /EPS_H1-49
- net /EPS_H1-52 renamed /EPS_H1-51
- net /EPS_H2-26 renamed /EPS_H2-25
- net /EPS_H2-28 renamed /EPS_H2-27
- net /H2-36 renamed /H2-35
- C6 pad 1: +5V -> /power/USB_VBUS
- IC1 pad 1: +5V -> /power/USB_VBUS
- R43 pad 2: /power/USB_VBUS -> +5V
Routing:
- net /H2-28: track 1205.2 -> 838.5 mm, vias 10 -> 7
- net /H2-26: track 1208.1 -> 844.6 mm
- net /H2-35: track 1169.2 -> 832.7 mm
- net /H1-46: track 1159.6 -> 852.9 mm, vias 13 -> 10
- net /H1-48: track 1134.4 -> 832.0 mm, vias 13 -> 10
- net /H1-52: track 1084.6 -> 789.7 mm, vias 9 -> 6
- net /H1-50: track 1109.8 -> 816.6 mm, vias 13 -> 10
- net /power/USB_VBUS: track 46.2 -> 131.2 mm
- net /H1_P: track 886.6 -> 899.1 mm, vias 6 -> 5
- net /SCL_CHN_3: track 636.7 -> 647.5 mm
- net /SDA_CHN_3: track 661.1 -> 670.9 mm
- net /H2_N: track 815.3 -> 823.2 mm, vias 7 -> 8
- net /H1_N: track 883.7 -> 879.4 mm, vias 6 -> 5
- net /microzed/<NO NET>: track 109.8 -> 113.1 mm
- net /H2_P: track 819.8 -> 822.8 mm
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