File: hardware/convert_folder/sources/power_schematic.kicad_sch (KiCad schematic)
At the start: 51 parts, among them CN1 5-146285-2, CN10 5-146285-2, CN13 4243-0, CN15 JST 2 position header 2.5mm, CN16 JST 2 position header 2.5mm, CN2 4243-0, CN3 4 pin Picoblade, CN8 5-146285-2, CN9 5-146285-2, IC1 TPS74401RGWRM3, IC2 TPS74401RGWRM3, IC4 TPS3899DL30DSER, IC5 LM321LVIDBVR, J3 1054500101, J8 87832-1420, J9 87832-1420, SW1 434123050836

Commit message: fix: fix a lot of connections between blocks. Many more to go...
Changed lines of the file:
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@@
 	)
 	(label "V2_E"
-		(at 407.67 104.14 0)
+		(at 412.75 104.14 0)
 		(effects
 			(font
@@
 	)
 	(label "V1_E"
-		(at 405.13 58.42 0)
+		(at 410.21 58.42 0)
 		(effects
 			(font

Commit message: fix: convert 90% of the schematic (there are 21 warnings/errors to resolve)
Parts:
- removed C11: CL10B104KA8NNNC, C0603_MD, symbol Capacitor:root_2_CL10B104KA8NNNC_Capacitor.SchLib
- removed C12: CL10B103KB8NNNC, C0603_MD, symbol Capacitor:root_0_CL10B103KB8NNNC_Capacitor.SchLib
- removed C13, C8: Cin, C0603_MD, symbol Capacitor:root_0_UMK107BJ105KA-T_Capacitor.SchLib
- removed C27, C5: Cout, C0603_MD, symbol Capacitor:root_0_GRM188C81C106MA73D_Capacitor.SchLib
- removed C52: CL10B473KB8NNNC, C0603_MD, symbol Capacitor:root_3_CL10B473KB8NNNC_Capacitor.SchLib
- removed C53: CL10B223KB8NNNC, C0603_MD, symbol Capacitor:root_3_CL10B223KB8NNNC_Capacitor.SchLib
- removed C54, C9: Cbias, C0603_MD, symbol Capacitor:root_0_UMK107BJ105KA-T_Capacitor.SchLib
- removed C55: CL10B103KB8NNNC, C0603_MD, symbol Capacitor:root_2_CL10B103KB8NNNC_Capacitor.SchLib
- removed C6: EMK107F105ZA-T, C0603_MD, symbol Capacitor:root_0_EMK107F105ZA-T_Capacitor.SchLib
- removed C7: CL10B104KA8NNNC, C0603_MD, symbol Capacitor:root_0_CL10B104KA8NNNC_Capacitor.SchLib
- removed CH1: Solder Jumper, Solder Jumper, symbol Miscellaneous:root_0_Solder Jumper_Miscellaneous.SchLib
- removed D1: ESDS314DBVR, C__Users_icaro_Desktop_SpaceLab_FlatSat_flatsat-platform2-hardware_hardware_libraries_flatsat_platform_2.PcbLib:SOT95P2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, symbol *:root_0_ESDS314DBVR_*
- removed IC1, IC2: TPS74401RGWRM3, C__Users_icaro_Documents_AltiumLL_SamacSys.PcbLib:QFN65P500X500X100-21N-D, symbol SamacSys:root_0_TPS74401RGWRM3_SamacSys.SchLib
- removed IC4: TPS3899DL30DSER, C__Users_icaro_Desktop_SpaceLab_FlatSat_flatsat-platform2-hardware_hardware_libraries_flatsat_platform_2.PcbLib:TPS3899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, symbol *:root_0_TPS3899DL30DSER_*
- removed IC5: LM321LVIDBVR, C__Users_icaro_Desktop_SpaceLab_FlatSat_flatsat-platform2-hardware_hardware_libraries_flatsat_platform_2.PcbLib:SOT95P2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, symbol *:root_0_LM321LVIDBVR_*
- removed LED1: 150160GS73103, 0603 (1608 metric), symbol flatsat_platform_2:root_0_150160GS73103_flatsat_platform_2.SchLib
- removed R1: RMCF0603FT47K0, R0603_HD, symbol Resistor:root_1_RMCF0603FT47K0_Resistor.SchLib
- removed R15: RMCF0603FT47K0, R0603_MD, symbol Resistor:root_0_RMCF0603FT47K0_Resistor.SchLib
- removed R2: ERJ-PB3B2492V, R0603_HD, symbol SamacSys:root_1_ERJ-PB3B2492V_SamacSys.SchLib
- removed R3: ERJH3ED3652V, R0603_HD, symbol SamacSys:root_1_ERJH3ED3652V_SamacSys.SchLib
- removed R4: ERJ-H3ED3652V, R0603_HD, symbol SamacSys:root_1_ERJ-H3ED3652V_SamacSys.SchLib
- removed R41: RC0603FR-07240RL, R0603_MD, symbol Resistor:root_1_RC0603FR-07240RL_Resistor.SchLib
- removed R5, R9: RMCF0603FT3K57, R0603_MD, symbol Resistor:root_0_RMCF0603FT3K57_Resistor.SchLib
- removed R6: CPF0603F1K15C1, R0603_MD, symbol SamacSys:root_0_CPF0603F1K15C1_SamacSys.SchLib
- removed S4: NDS02V, C__Users_icaro_Documents_AltiumLL_SamacSys.PcbLib:NDS02V, symbol SamacSys:root_0_NDS02V_SamacSys.SchLib
- removed SW1: 434123050836, 4341x30508x6, symbol Switch:root_3_434123050836_Switch.SchLib
- C1: footprint C0603_MD -> altium_import:C0603_MD; symbol Capacitor:root_0_GRM188R71C103KA01D_Capacitor.SchLib -> altium_import:root_0_GRM188R71C103KA01D_Capacitor.SchLib
- C2: footprint C0603_MD -> altium_import:C0603_MD; symbol Capacitor:root_0_CL10B104KA8NNNC_Capacitor.SchLib -> altium_import:root_0_CL10B104KA8NNNC_Capacitor.SchLib
- C20: footprint C__Users_icaro_Documents_AltiumLL_SamacSys.PcbLib:CAPAE660X770N -> altium_import:CAPAE660X770N; symbol *:root_3_865080845004_* -> altium_import:root_3_865080845004_*
- C3: footprint C0603_MD -> altium_import:C0603_MD; symbol Capacitor:root_0_GRM188R71H104JA93D_Capacitor.SchLib -> altium_import:root_0_GRM188R71H104JA93D_Capacitor.SchLib
- C4: footprint C0603_MD -> altium_import:C0603_MD; symbol Capacitor:root_0_EMK107BB7225MA-T_Capacitor.SchLib -> altium_import:root_0_EMK107BB7225MA-T_Capacitor.SchLib
- CN1, CN10, CN8, CN9: footprint PIN BAR 2 2.54mm 180 GRAUS -> altium_import:PIN BAR 2 2.54mm 180 GRAUS; symbol Connector:root_2_5-146285-2_Connector.SchLib -> altium_import:root_2_5-146285-2_Connector.SchLib_1
- CN13, CN2: footprint 4243-0 -> altium_import:4243-0; symbol flatsat_platform_2:root_1_4243-0_flatsat_platform_2.SchLib -> altium_import:root_1_4243-0_flatsat_platform_2.SchLib
- CN15: footprint B2B-XH-A-M(LF)(SN) -> altium_import:B2B-XH-A-M(LF)(SN); symbol Connector:root_2_5-146285-2_Connector.SchLib -> altium_import:root_2_5-146285-2_Connector.SchLib
- CN16: footprint B2B-XH-A-M(LF)(SN) -> altium_import:B2B-XH-A-M(LF)(SN); symbol flatsat_platform_2:root_0_mirrored_B2B-XH-A-M(LF)(SN)_flatsat_platform_2.SchLib -> altium_import:root_0_mirrored_B2B-XH-A-M(LF)(SN)_flatsat_platform_2.SchLib
- CN3: footprint PICO BLADE 0532610471 -> altium_import:PICO BLADE 0532610471; symbol flatsat_platform_2:root_2_mirrored_0533980471_flatsat_platform_2.SchLib -> altium_import:root_2_mirrored_0533980471_flatsat_platform_2.SchLib
- J3: footprint FP-1054500101-MFG -> altium_import:FP-1054500101-MFG; symbol Altium Content Vault:root_0_9808b19ecaf079fb99eed69f0495cd0_Altium Content Vault -> altium_import:root_0_9808b19ecaf079fb99eed69f0495cd0_Altium Content Vault
- J8, J9: footprint SAMTEC_TSW-107-05-F-D -> altium_import:SAMTEC_TSW-107-05-F-D; symbol flatsat_platform_2:root_3_87832-1420_flatsat_platform_2.SchLib -> altium_import:root_3_87832-1420_flatsat_platform_2.SchLib
- L1: footprint C__Users_icaro_Documents_AltiumLL_SamacSys.PcbLib:WE-PF_7427929...60 -> altium_import:WE-PF_7427929...60; symbol SamacSys:root_0_742792901_SamacSys.SchLib -> altium_import:root_0_742792901_SamacSys.SchLib
- R10, R11: footprint R0603_MD -> altium_import:R0603_MD; symbol Resistor:root_1_RMCF0603FT5K10_Resistor.SchLib -> altium_import:root_1_RMCF0603FT5K10_Resistor.SchLib
Connections:
- net VBAT: now also CN16.1
- no-connect marks 19 -> 18
Other:
- added sheet fixed-3v3-converter (fixed-3v3-converter.kicad_sch)
- added sheet fixed-3v3-converter1 (fixed-3v3-converter.kicad_sch)
- added sheet non-fixed-voltage-converter (non-fixed-voltage-converter.kicad_sch)
- added sheet non-fixed-voltage-converter1 (non-fixed-voltage-converter.kicad_sch)
- note removed: "1V8"
- note removed: "2V5"
- note removed: "3V3"
- note removed: "ADJ selectable voltage divider (ADJ=0.8V)"
- note removed: "DECAPS"
- moved on the sheet: CN15, CN3

Commit message: fix: start fixing the power converters of the board
Parts:
- removed C3: GRM188R71H104JA93D, altium_import:C0603_MD, symbol altium_import:root_0_GRM188R71H104JA93D_Capacitor.SchLib
- removed C4: EMK107BB7225MA-T, altium_import:C0603_MD, symbol altium_import:root_0_EMK107BB7225MA-T_Capacitor.SchLib
- removed CN10: 5-146285-2, altium_import:PIN BAR 2 2.54mm 180 GRAUS, symbol altium_import:root_2_5-146285-2_Connector.SchLib_1
- removed CN16: JST 2 position header 2.5mm, altium_import:B2B-XH-A-M(LF)(SN), symbol altium_import:root_0_mirrored_B2B-XH-A-M(LF)(SN)_flatsat_platform_2.SchLib
- added C6: GRM188R71H104JA93D, altium_import:C0603_MD, symbol altium_import:root_0_GRM188R71H104JA93D_Capacitor.SchLib
- added CN11, CN7: 5-146285-2, altium_import:PIN BAR 2 2.54mm 180 GRAUS, symbol altium_import:root_2_5-146285-2_Connector.SchLib_1
- added IC1: TPS3780BDBVT, lib:TPS3780BDBVT, symbol lib:TPS3780BDBVT
- added R15, R23, R24, R32, R33, R34: DNP, altium_import:0805, symbol altium_import:RDNP_0805
Connections:
- net +5V: now also C6.1, IC1.1 (VDD), R24.1, R33.1; no longer CN9.1
- net GND: now also CN1.1, CN8.1, CN9.1, C6.2, CN11.1, CN7.1, IC1.5 (GND), R32.2, R34.2
- net VCCIO_{13}: now also CN11.2
- net VCCIO_{34}: now also CN7.2
- net VS: no longer CN1.1
- net VCCIO renamed VCCIO_{35}
- net VCCIO_{35}: no longer CN8.1
- new net: IC1.2 (OUT1), R23.2
- new net: IC1.6 (SENSE1), R33.2, R34.1
- new net: IC1.4 (SENSE2), R24.2, R32.1
- new net: IC1.3 (OUT2), R15.2
- new net PWR_EN: R23.1
- new net VCCIO_EN: R15.1
Other:
- sheet fixed-3v3-converter renamed fixed-VS-converter
- sheet fixed-3v3-converter1 renamed fixed-bank-13-converter
- sheet non-fixed-voltage-converter renamed non-fixed-bank-34-converter
- sheet non-fixed-voltage-converter1 renamed non-fixed-bank-35-converter
- moved on the sheet: C1, C2, C20, CN1, CN9, J3A, J3B, J3C, L1, R10, R11

Commit message: fix: add more fixes to the power converters, add resets and other minor corrections
Parts:
- added R39: DNP, altium_import:0805, symbol altium_import:RDNP_0805
- added TP12, TP13: ~, altium_import:TEST POINT PTH, symbol altium_import:root_0_Test Point PTH_flatsat_platform_2.SchLib
Connections:
- net GND: now also R39.1
- net V1_E: now also TP12.1
- net V2_E: now also TP13.1
- net at J3.1 (MNT_1): now also J3.2 (MNT_2), J3.3 (MNT_3), J3.4 (MNT_4), R39.2
- no-connect marks 18 -> 14
Other:
- sheet fixed-VS-converter ports: added PG_CARRIER, VCCIO_EN; removed none
- sheet fixed-bank-13-converter ports: added PG_CARRIER, VCCIO_EN; removed none
- sheet non-fixed-bank-34-converter ports: added PG_CARRIER, VCCIO_EN; removed none
- sheet non-fixed-bank-35-converter ports: added PG_CARRIER, VCCIO_EN; removed none

Commit message: fix: start the layout of power path
Parts:
- added TP11, TP4: ~, altium_import:TEST POINT PTH, symbol altium_import:root_0_Test Point PTH_flatsat_platform_2.SchLib
Connections:
- net +5V: now also TP4.1
- net VS: now also TP11.1

Commit message: chore: add minor modifications do the layout
Parts:
- removed J3: 1054500101, altium_import:FP-1054500101-MFG, symbol altium_import:root_0_9808b19ecaf079fb99eed69f0495cd0_Altium Content Vault
- removed R10, R11: RMCF0603FT5K10, altium_import:R0603_MD, symbol altium_import:root_1_RMCF0603FT5K10_Resistor.SchLib
- removed R39: DNP, altium_import:0805, symbol altium_import:RDNP_0805
- added D1: LED, LED_SMD:LED_0603_1608Metric, symbol Device:LED
- added J3: USB-C, altium_import:FP-1054500101-MFG, symbol connectors:USB-C
- added R41, R42: 5.11k, footprints:RES0402, symbol resistors:CRCW04025K11FKED
- added R43: 1k, footprints:RES0603, symbol resistors:CRCW06031K00FKEAHP
Connections:
- net GND: now also D1.1 (K), J3.A1 (GND), J3.A12 (GND), J3.B1 (GND), J3.B12 (GND), J3.S1 (SHIELD), R41.1, R42.1
- net USB_VBUS: now also J3.A4 (VBUS), J3.A9 (VBUS), J3.B4 (VBUS), J3.B9 (VBUS), R43.2
- new net: J3.B5 (CC2), R41.2
- new net: J3.A5 (CC1), R42.2
- new net: D1.2 (A), R43.1
- no-connect marks 14 -> 6
Other:
- note added: "Improve the input power circuitry of the project, something similar to what is presented, for instance, in:"
- note added: "Update for the future:"
- note added: "https://resources.altium.com/p/add-usb-type-c-power-delivery-your-designs"
- moved on the sheet: C1, C2, C20, CN9, L1, TP4

Commit message: fix: improve CAN-related routing and other minor layout-related things
Parts:
- added SW1: SW-T3-2B-A-A3-S1, altium_import:SW-T3-2B-A-A3-S1, symbol altium_import:root_2_SW-T3-2B-A-A3-S1_SW-T3-2B-A-A3-S1.SchLib
Connections:
- net USB_VBUS: now also SW1.2 (COM); no longer C1.1, L1.1
- new net: C1.1, L1.1, SW1.3
- no-connect marks 6 -> 7
Changed lines of the file:
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@@
+	)
+	(no_connect
+		(at 228.6 124.46)
 	)
 	(no_connect
@@
 	(wire
 		(pts
+			(xy 210.82 127) (xy 213.36 127)
+		)
+		(stroke
+			(width 0.381)
+			(type default)
+		)
+	)
+	(wire
+		(pts
 			(xy 36.83 237.49) (xy 54.61 237.49)
 		)
@@
 	(wire
 		(pts
-			(xy 237.49 129.54) (xy 222.25 129.54)
+			(xy 237.49 129.54) (xy 228.6 129.54)
 		)
 		(stroke
@@
 	)
 	(label "USB_VBUS"
-		(at 222.25 129.54 0)
-		(effects
-			(font
-				(size 1.27 1.27)
-			)
-			(justify left bottom)
+		(at 210.82 127 180)
+		(effects
+			(font
+				(size 1.27 1.27)
+			)
+			(justify right bottom)
 		)
 	)
@@
 					(unit 1)
 				)
+			)
+		)
+	)
+	(symbol
+		(lib_id "altium_import:root_2_SW-T3-2B-A-A3-S1_SW-T3-2B-A-A3-S1.SchLib")
+		(at 223.52 127 90)
+		(unit 1)
+		(exclude_from_sim no)
+		(in_bom yes)
+		(on_board yes)
+		(dnp no)
+		(property "Reference" "SW1"
+			(at 226.314 130.302 90)
+			(effects
+				(font
+					(size 1.27 1.27)
+				)
+				(justify left bottom)
+			)
+		)
+		(property "Value" "SW-T3-2B-A-A3-S1"
+			(at 226.314 121.158 90)
+			(effects
+				(font
+					(size 1.27 1.27)
+				)
+				(justify left bottom)
+			)
+		)
+		(property "Footprint" "altium_import:SW-T3-2B-A-A3-S1"
+			(at 223.52 127 0)
+			(effects
+				(font
+					(size 1.27 1.27)
+				)
+				(hide yes)
+			)
+		)
+		(property "Datasheet" ""
+			(at 223.52 127 0)
+			(effects
+				(font
+					(size 1.27 1.27)
+				)
+				(hide yes)
+			)
+		)
+		(property "Description" "SW-T3-2B-A-A3-S1"
+			(at 223.52 127 0)
+			(effects
+				(font
+					(size 1.27 1.27)
+				)
+				(hide yes)
+			)
+		)
+		(pin "2"
+		)
+		(pin "1"
+		)
+		(pin "3"
+		)
+		(instances
+			(project "flatsat_platform_2"
+				(path "/8c88a7e1-4137-48d7-b926-b5e762e3852f/8386d232-e6d5-4b15-8289-83f2ee4d46fe"
+					(reference "SW1")
+					(unit 1)
+				)
