File: hardware/convert_folder/sources/microzed_schematic.kicad_sch (KiCad schematic)
At the start: 15 parts, among them J20 61201421621, J21 61201421621

Commit message: fix: fix caps. values, add decoupling capacitors for INAs and other ICs, and add general improvements
Parts:
- removed R40, R47: DNP, altium_import:0805, symbol altium_import:RDNP_0805
- added R7, R8: 2.2k, lib:RES0805, symbol resistors:CRCW08052K20FKEAHP
Connections:
- net P2: now also SOM1.JX1-9 (JX1_SE_0); no longer SOM1.JX1-11 (JX1_LVDS_0_P)
- net P4: now also SOM1.JX1-11 (JX1_LVDS_0_P); no longer SOM1.JX1-13 (JX1_LVDS_0_N)
- net P6: now also SOM1.JX1-13 (JX1_LVDS_0_N); no longer SOM1.JX1-17 (JX1_LVDS_2_P)
- net SCL_CHN_3: now also R7.2
- net SDA_CHN_3: now also R8.2
- net VS: now also R7.1, R8.1
- net PL_JX2_17P: now reaches J21.12, SOM1.JX2-68 (JX2_LVDS_17_P)
