File: hardware/convert_folder/sources/voltage_level_translators_schematic.kicad_sch (KiCad schematic)
At the start: 48 parts, among them CN14 TSW-101-05-T-S, IC6 MMBT3904, IC7 MMBT3904, J1 5-146280-2, J10 Soquete de termopar, J11 Soquete de termopar, J12 Soquete de termopar, J13 Soquete de termopar, J14 Soquete de termopar, J15 Soquete de termopar, J2 5-146280-2, J5 Soquete de termopar, J6 Soquete de termopar, M1 IB Mechanical Hole, M2 IB Mechanical Hole, M3 IB Mechanical Hole, M4 IB Mechanical Hole, U1 INA219AID, U12 INA219AID, U13 INA219AID, U18 INA219AID, U19 TMP112AIDRLT, U21 LTC2983CLX#PBF, U22 ISL83483IBZ, U25 ISL83483IBZ, U4 INA219AID, U7 INA219AID, U9 INA219AID

Commit message: fix: fix a lot of connections between blocks. Many more to go...
Other:
- note removed: "RS485 bidirectional voltage-level translator"

Commit message: fix: convert 90% of the schematic (there are 21 warnings/errors to resolve)
Parts:
- removed C14, C15: 1.0uF/50V, CC0805, symbol flatsat_platform_2:root_1_Cap_Cer_X7R_1.0uF_50V_0805_flatsat_platform_2.SchLib
- removed C16, C17, C18: 10uF/16V, CC1210, symbol flatsat_platform_2:root_1_Cap_Cer_X7R_10uF_16V_1210_flatsat_platform_2.SchLib
- removed C19, C21, C22, C23, C24, C25, C26, C28: 0.1uF/25V, CC0805, symbol flatsat_platform_2:root_1_Cap_Cer_X7R_0.1uF_25V_0805_flatsat_platform_2.SchLib
- removed CN14: TSW-101-05-T-S, PIN BAR 1 2.54mm 180 GRAUS - Hide, symbol flatsat_platform_2:root_2_TSW-101-05-T-S_flatsat_platform_2.SchLib
- removed IC6, IC7: MMBT3904, C__Users_icaro_Documents_AltiumLL_SamacSys.PcbLib:SOT95P240X120-3N, symbol *:root_0_MMBT3904_*
- removed J10, J11, J12, J13, J14, J15, J5, J6: Soquete de termopar, PCC-SMP-V-K, symbol Thermocouple_connector:root_0_PCC-SMP-V-K_Thermocouple_connector.SchLib
- removed M1, M2, M3, M4: IB Mechanical Hole, M3 hole (5.5mm pad), symbol iip:root_0_IB Mechanical Hole_iip.SchLib
- removed U1, U12, U13, U18, U4, U7, U9: INA219AID, SOIC127P599X175-8N, symbol flatsat_platform_2:root_0_INA219AID_flatsat_platform_2.SchLib
- removed U21: LTC2983CLX#PBF, QFP50P900X900X160-48N, symbol flatsat_platform_2:root_0_LTC2983CLX#PBF_flatsat_platform_2.SchLib
- added NT1, NT2, NT3, NT4, NT5, NT6, NT7: NetTie_2, symbol Device:NetTie_2
- added U1, U12, U13, U18, U4, U7, U9: INA219AID, altium_import:SOIC127P599X175-8N, symbol altium_import:root_0_INA219AID_flatsat_platform_2.SchLib
- J1, J2: footprint PIN BAR 2 2.54mm 180 GRAUS -> altium_import:PIN BAR 2 2.54mm 180 GRAUS; symbol flatsat_platform_2:root_0_5-146280-2_flatsat_platform_2.SchLib -> altium_import:root_0_5-146280-2_flatsat_platform_2.SchLib
- R25, R26, R27, R28, R29, R30, R31: footprint 0805 -> altium_import:0805; symbol flatsat_platform_2:root_2_RDNP_0805_flatsat_platform_2.SchLib -> altium_import:RDNP_0805
- U19: footprint SOT50P160X60-6N -> altium_import:SOT50P160X60-6N; symbol flatsat_platform_2:root_0_TMP112AIDRLT_flatsat_platform_2.SchLib -> altium_import:root_0_TMP112AIDRLT_flatsat_platform_2.SchLib; ALTIUM_VALUE * -> (none); AVAILABILITY Good -> (none); DIGIKEY-PURCHASE-URL https://snapeda.com/shop?store=DigiKey&id=237309 -> (none); MANUFACTURER PART NUMBER TMP112AIDRLT -> (none); MF Texas Instruments -> (none); MOUSER-PURCHASE-URL https://snapeda.com/shop?store=Mouser&id=237309 -> (none); PACKAGE SOT-5X3-6 Texas Instruments -> (none); PRICE None -> (none); SNAPEDA_LINK https://www.snapeda.com/parts/TMP112AIDRLT/Texas%20Instrume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 -> (none); TEXAS_INSTRUMENTS-PURCHASE-URL https://snapeda.com/shop?store=Texas+Instruments&id=237309 -> (none)
- U22, U25: footprint SOIC127P600X175-8N -> altium_import:SOIC127P600X175-8N; symbol flatsat_platform_2:root_0_ISL83483IBZ_flatsat_platform_2.SchLib -> altium_import:root_0_ISL83483IBZ_flatsat_platform_2.SchLib; ALTIUM_VALUE * -> (none); AVAILABILITY Unavailable -> (none); MANUFACTURER PART NUMBER ISL83483IBZ-T -> (none); MF Renesas Electronics -> (none); PACKAGE SOIC-8 Intersil -> (none); PRICE None -> (none); SNAPEDA_LINK https://www.snapeda.com/parts/ISL83483IBZ-T/Renesas%20Elect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 -> (none)
Connections:
- net EPS_H1-45: now also NT1.1, U1.8 (VIN+)
- net EPS_H1-47: now also NT3.1, U4.8 (VIN+)
- net EPS_H1-49: now also NT2.1, U7.8 (VIN+)
- net EPS_H1-51: now also NT4.1, U9.8 (VIN+)
- net EPS_H2-25: now also NT6.2; no longer R30.1
- net EPS_H2-27: now also NT7.2; no longer R31.1
- net EPS_H2-35: now also NT5.1, U12.8 (VIN+)
- net GND: now also U1.1 (A1), U1.2 (A0), U1.6 (GND), U12.2 (A0), U12.6 (GND), U13.6 (GND), U18.6 (GND), U4.1 (A1), U4.6 (GND), U7.1 (A1), U7.6 (GND), U9.1 (A1), U9.6 (GND)
- net H1-45: now also U1.7 (VIN-)
- net H1-47: now also U4.7 (VIN-)
- net H1-49: now also U7.7 (VIN-)
- net H1-51: now also U9.7 (VIN-)
- net H2-25: now also U13.7 (VIN-)
- net H2-27: now also U18.7 (VIN-)
- net H2-35: now also U12.7 (VIN-)
- net SCL_CHN_3: now also U1.4 (SCL), U12.4 (SCL), U13.4 (SCL), U18.4 (SCL), U4.4 (SCL), U7.2 (A0), U7.4 (SCL), U9.4 (SCL)
- net SDA_CHN_3: now also U1.3 (SDA), U12.3 (SDA), U13.3 (SDA), U18.2 (A0), U18.3 (SDA), U4.3 (SDA), U7.3 (SDA), U9.2 (A0), U9.3 (SDA)
- net VS: now also U1.5 (VS), U12.1 (A1), U12.5 (VS), U13.1 (A1), U13.2 (A0), U13.5 (VS), U18.1 (A1), U18.5 (VS), U4.2 (A0), U4.5 (VS), U7.5 (VS), U9.5 (VS)
- new net EPS_H1-46: NT1.2
- new net EPS_H1-48: NT3.2
- new net EPS_H1-50: NT2.2
- new net EPS_H1-52: NT4.2
- new net EPS_H2-26: NT6.1, R30.1, U13.8 (VIN+)
- new net EPS_H2-28: NT7.1, R31.1, U18.8 (VIN+)
- new net EPS_H2-36: NT5.2
- no-connect marks 9 -> 1
Other:
- note removed: "Cold Junction Measurement"
- note removed: "Components temperature measurement system"
- note removed: "Interface Board Mechanical Holes"
- moved on the sheet: R25, R26, R27, R28, R29, R30, R31

Commit message: fix: add more fixes to the power converters, add resets and other minor corrections
Changed lines of the file:
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@@
 	(wire
 		(pts
-			(xy 544.83 232.41) (xy 552.45 232.41)
-		)
-		(stroke
-			(width 0)
-			(type default)
-		)
-	)
-	(wire
-		(pts
 			(xy 267.97 52.07) (xy 262.89 52.07)
 		)
@@
 	(wire
 		(pts
+			(xy 544.83 232.41) (xy 552.45 232.41)
+		)
+		(stroke
+			(width 0)
+			(type default)
+		)
+	)
+	(wire
+		(pts
 			(xy 87.63 213.36) (xy 80.01 213.36)
 		)
@@
 		(dnp no)
 		(property "Reference" "R30"
-			(at 62.484 318.262 90)
+			(at 62.23 310.388 90)
 			(effects
 				(font
@@
 		)
 		(property "Value" "DNP"
-			(at 59.944 318.262 90)
+			(at 59.69 310.388 90)
 			(effects
 				(font

Commit message: fix: start the layout of power path
Parts:
- removed NT1, NT2, NT3, NT4, NT5, NT6, NT7: NetTie_2, symbol Device:NetTie_2
- removed U22, U25: ISL83483IBZ, altium_import:SOIC127P600X175-8N, symbol altium_import:root_0_ISL83483IBZ_flatsat_platform_2.SchLib
- added U22, U25: THVD1450DR, lib:THVD1450DR, symbol lib:THVD1450DR
Connections:
- net EPS_H2-26 is gone; now on net EPS_H2-25: R30.1, U13.8 (VIN+)
- net EPS_H2-28 is gone; now on net EPS_H2-27: R31.1, U18.8 (VIN+)
- net GND: now also U22.5 (GND), U25.5 (GND)
- net RS485_01_N: now also U22.6 (A)
- net RS485_01_P: now also U22.7 (B)
- net RS485_02_N: now also U25.6 (A)
- net RS485_02_P: now also U25.7 (B)
- net RX_CHN_3: now also U22.4 (D)
- net RX_CHN_4: now also U25.4 (D)
- net T/R_CHN_3: now also U22.1 (R), U22.3 (DE)
- net T/R_CHN_4: now also U25.1 (R), U25.3 (DE)
- net TX_CHN_3: now also U22.2 (~{RE})
- net TX_CHN_4: now also U25.2 (~{RE})
- net VS: now also U22.8 (VCC), U25.8 (VCC)
Other:
- moved on the sheet: J1, J2

Commit message: fix: fix some footprints and the position of refs. in the layout
Connections:
- net RX_CHN_3: now also U22.1 (R); no longer U22.4 (D)
- net RX_CHN_4: now also U25.1 (R); no longer U25.4 (D)
- net T/R_CHN_3: now also U22.2 (~{RE}); no longer U22.1 (R)
- net T/R_CHN_4: now also U25.2 (~{RE}); no longer U25.1 (R)
- net TX_CHN_3: now also U22.4 (D); no longer U22.2 (~{RE})
- net TX_CHN_4: now also U25.4 (D); no longer U25.2 (~{RE})

Commit message: fix: fix caps. values, add decoupling capacitors for INAs and other ICs, and add general improvements
Parts:
- added C42, C43, C44, C45, C46, C47, C48, C49, C50, C51: 100nF, lib:CAP0603, symbol capacitors:C0603C104K5RACTU
- added R33, R34, R40, R44: 10k, lib:RES0603, symbol resistors:CRCW060310K0FKEAHP
- added R47, R48: 120R, lib:RES0603, symbol resistors:CRCW0603120RFKEAHP
- R25, R26, R27, R28, R29, R30, R31: value DNP -> 47m
Connections:
- net GND: now also C42.1, C43.1, C44.1, C45.1, C46.1, C47.1, C48.1, C49.1, C50.1, C51.1, R33.1, R34.2
- net RS485_01_N: now also J2.1, U22.7 (B), R48.1; no longer J2.2, U22.6 (A)
- net RS485_01_P: now also J2.2, U22.6 (A), R48.2; no longer J2.1, U22.7 (B)
- net RS485_02_N: now also J1.1, U25.7 (B), R47.1; no longer J1.2, U25.6 (A)
- net RS485_02_P: now also J1.2, U25.6 (A), R47.2; no longer J1.1, U25.7 (B)
- net RX_CHN_3: now also R44.1
- net RX_CHN_4: now also R40.1
- net T/R_CHN_3: now also R33.2
- net T/R_CHN_4: now also R34.1
- net VS: now also C42.2, C43.2, C44.2, C45.2, C46.2, C47.2, C48.2, C49.2, C50.2, C51.2, R40.2, R44.2
Other:
- moved on the sheet: J1, J2, U22, U25
